Commit message: update kinetic source code

File: 3.Sofrware&Firmware/Leizhuo_UnderWaterHexapodRobot/urdf/Leizhuo_UnderWaterHexapodRobot.urdf (robot description, URDF)
Before this commit: robot Leizhuo_UnderWaterHexapodRobot, 37 links, 36 joints
Joints:
- removed joint RM_P_LINK
- added joint RM_P_JOINT: type revolute, parent RM_R_LINK, child RM_P_LINK, origin xyz=0 0 0 rpy=0 1.5708 0, axis 0 0 -1, limit lower=-1.5708 upper=1.5708 effort=0 velocity=0
